File: PCB/SOS_Schematic (5).kicad_sch (KiCad schematic)
At the start: 47 parts, among them J1 629722000214, J3 Conn_01x08, SW1 SW_SPDT, SW2 SW_Push, SW3 SW_Push, SW4 SW_Push, SW5 SW_Push, U1 BU33SD5WG-TR, U2 USBLC6-2SC6, U3 STM32L476RGTx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

Commit message: PCB final
Connections:
- net GND: now also J3.1 (Pin_1), U2.1 (I/O1); no longer J3.4 (Pin_4), U2.2 (GND)
- net RFID_IRQ: now also J3.4 (Pin_4); no longer J3.1 (Pin_1)
- net RFID_RST: now also J3.3 (Pin_3); no longer J3.5 (Pin_5)
- net SPI1_MISO: now also J3.5 (Pin_5); no longer J3.7 (Pin_7)
- net SPI1_MOSI: now also J3.2 (Pin_2); no longer J3.6 (Pin_6)
- net SPI1_NSS: now also J3.7 (Pin_7); no longer J3.2 (Pin_2)
- net SPI1_SCK: now also J3.6 (Pin_6); no longer J3.3 (Pin_3)
- net USBDP: now also U2.2 (GND); no longer U2.1 (I/O1)
