File: PCB/_autosave-SOS_Schematic (5).kicad_pcb (KiCad board)
At the start: 4 copper layers, 96 x 96 mm, 47 parts, among them J1 629722000214, J3 Conn_01x08, SW1 SW_SPDT, SW2 SW_Push, SW3 SW_Push, SW4 SW_Push, SW5 SW_Push, U1 BU33SD5WG-TR, U2 USBLC6-2SC6, U3 STM32L476RGTx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

Commit message: Dernière version
Other:
- board text added: "B"
- board text added: "Projet SOS"
- board text added: "T"
Changed lines of the file:
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@@
 		(layer "Edge.Cuts")
+	)
+	(gr_text "Projet SOS"
+		(at 169 122 0)
+		(layer "F.Cu")
+		(effects
+			(font
+				(size 1 1)
+				(thickness 0.15)
+			)
+			(justify left bottom)
+		)
+	)
+	(gr_text "T"
+		(at 140 54 0)
+		(layer "F.Cu")
+		(effects
+			(font
+				(size 2 2)
+				(thickness 0.5)
+				(bold yes)
+			)
+			(justify left bottom)
+		)
+	)
+	(gr_text "B"
+		(at 135 52 180)
+		(layer "B.Cu")
+		(effects
+			(font
+				(size 2 2)
+				(thickness 0.5)
+				(bold yes)
+			)
+			(justify left bottom mirror)
+		)
 	)
 	(segment
