File: Hardware/SOS_Schematic.kicad_sch (KiCad schematic)
At the start: 47 parts, among them J1 629722000214, J3 Conn_01x08, SW1 SW_SPDT, SW2 SW_Push, SW3 SW_Push, SW4 SW_Push, SW5 SW_Push, U1 BU33SD5WG-TR, U2 USBLC6-2SC6, U3 STM32L476RGTx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

Commit message: review pcb
Parts:
- added C16: 100n, Capacitor_SMD:C_0402_1005Metric, symbol Device:C_Small
- C1, C10, C11, C14, C2, C5, C7, C8, C9: footprint Capacitor_SMD:C_0603_1608Metric -> Capacitor_SMD:C_0402_1005Metric
- J2: value ~ -> (none)
- R1, R10, R11, R12, R2, R3, R4, R5, R7, R8, R9: footprint Resistor_SMD:R_0603_1608Metric -> Resistor_SMD:R_0402_1005Metric
- R6: footprint Button_Switch_SMD:SW_SPST_CK_KMS2xxG -> Resistor_SMD:R_0402_1005Metric
- SW1: footprint Button_Switch_THT:SW_Slide_SPDT_Straight_CK_OS102011MS2Q -> Button_Switch_SMD:SW_SPDT_CK_JS102011SAQN
Connections:
- net SWDCK is gone; now on net SWCLK: U3.49 (PA14)
- net +3.3V: now also C16.1
- net GND: now also J3.1 (Pin_1), C16.2; no longer J3.6 (Pin_6)
- net RFID_IRQ: now also J3.4 (Pin_4); no longer J3.1 (Pin_1)
- net RFID_RST: now also J3.3 (Pin_3); no longer J3.7 (Pin_7)
- net SPI1_MOSI: now also J3.2 (Pin_2); no longer J3.4 (Pin_4)
- net SPI1_NSS: now also J3.7 (Pin_7); no longer J3.2 (Pin_2)
- net SPI1_SCK: now also J3.6 (Pin_6); no longer J3.3 (Pin_3)
- net SWO: now also U3.55 (PB3)
- net BTN_0 renamed USR_BTN_1
- net BTN_1 renamed USR_BTN_2
- no-connect marks 37 -> 36
